Commit message: Remove unused scenes, split arm into separte configs for easier including, update default keyframe, remove duplicate joint state publisher from launch

File: src/site_configs/picknik_kinova_satellite_sim/description/picknik_kinova_satellite_sim.xacro (robot description, xacro)
@@ -4,29 +4,10 @@
     <xacro:arg name="arm" default="gen3" />
     <xacro:arg name="dof" default="7" />
-    <xacro:arg name="vision" default="false" />
-    <xacro:arg name="gripper" default="" />
-    <xacro:arg name="gripper_joint_name" default="robotiq_85_left_knuckle_joint" />
-    <xacro:arg name="use_internal_bus_gripper_comm" default="true" />
-    <xacro:arg name="prefix" default="" />
-    <xacro:arg name="use_fake_hardware" default="false" />
-    <xacro:arg name="fake_sensor_commands" default="false" />
-    <xacro:arg name="sim_gazebo" default="false" />
-    <xacro:arg name="sim_ignition" default="false" />
-    <xacro:arg name="sim_isaac" default="false" />
-    <xacro:arg name="isaac_joint_commands" default="/isaac_joint_commands" />
-    <xacro:arg name="isaac_joint_states" default="/isaac_joint_states" />
-    <xacro:arg name="use_external_cable" default="false" />
-    <xacro:arg name="gripper_max_velocity" default="100.0" />
-    <xacro:arg name="gripper_max_force" default="100.0" />
-    <xacro:arg name="gripper_com_port" default="/dev/ttyUSB0" />
-    <xacro:arg name="wrist_realsense" default="true" />
+    <xacro:arg name="mujoco_keyframe" default="default" />
     <xacro:arg name="mujoco_model" default="description/mujoco/scene.xml" />
     <xacro:arg name="mujoco_viewer" default="false" />
     <!-- Import macros for main hardware components -->
     <xacro:include filename="$(find kortex_description)/arms/$(arg arm)/$(arg dof)dof/urdf/$(arg arm)_macro.xacro" />
-    <!-- <xacro:include filename="$(find kortex_description)/grippers/$(arg gripper)/urdf/$(arg gripper)_macro.xacro" /> -->
     <xacro:include filename="$(find picknik_accessories)/descriptions/sensors/realsense_d415.urdf.xacro"/>
-    <!-- Import environment macros -->
-    <xacro:include filename="$(find picknik_accessories)/descriptions/geometry/cube.urdf.xacro"/>
     <!-- World is centered under base_link of the robot, on the ground -->
     <link name="world"/>
@@ -36,5 +17,5 @@
     <!-- Load the arm -->
     <joint name="base_joint" type="fixed">
-      <origin rpy="0 0 0" xyz="0 0 0.02"/>
+      <origin rpy="1.5708 0 1.5708" xyz="0 0 0.5"/>
       <parent link="world"/>
       <child link="base_link"/>
@@ -529,8 +510,4 @@
       <mimic joint="robotiq_85_left_knuckle_joint" multiplier="-1"/>
     </joint>
-    <!-- Environment -->
-    <xacro:cube link_name="table" connected_to="world" length="2.00" width="2.00" height="0.25" alpha="0.3">
-      <origin xyz="0 0 -0.145" rpy="0 0 0"/>
-    </xacro:cube>
     <!-- Visual aids for grasping -->
     <link name="finger_tip_closed_point">
@@ -561,5 +538,5 @@
       <parent link="world" />
       <child link="external_camera_link" />
-      <origin xyz="-0.3 0.3 1.0" rpy="0.0 0.4 0" />
+      <origin xyz="-0.3 0.3 1.0" rpy="0 0.5236 0" />
     </joint>
     <xacro:realsense_d415 parent="external_camera_link" name="scene_camera">
@@ -673,4 +650,5 @@
       <hardware>
         <plugin>picknik_mujoco_ros/MujocoSystem</plugin>
+        <param name="mujoco_keyframe">$(arg mujoco_keyframe)</param>
         <param name="mujoco_model">$(arg mujoco_model)</param>
         <param name="mujoco_model_package">picknik_kinova_satellite_sim</param>

Commit message: Add table back to xacro and return to vertical arm mount, update srdf and keyframes accordingly

File: src/site_configs/picknik_kinova_satellite_sim/description/picknik_kinova_satellite_sim.xacro (robot description, xacro)
@@ -10,4 +10,6 @@
     <xacro:include filename="$(find kortex_description)/arms/$(arg arm)/$(arg dof)dof/urdf/$(arg arm)_macro.xacro" />
     <xacro:include filename="$(find picknik_accessories)/descriptions/sensors/realsense_d415.urdf.xacro"/>
+    <!-- Import environment macros -->
+    <xacro:include filename="$(find picknik_accessories)/descriptions/geometry/cube.urdf.xacro"/>
     <!-- World is centered under base_link of the robot, on the ground -->
     <link name="world"/>
@@ -17,5 +19,5 @@
     <!-- Load the arm -->
     <joint name="base_joint" type="fixed">
-      <origin rpy="1.5708 0 1.5708" xyz="0 0 0.5"/>
+      <origin rpy="0 0 0" xyz="0 0 0.02"/>
       <parent link="world"/>
       <child link="base_link"/>
@@ -510,4 +512,8 @@
       <mimic joint="robotiq_85_left_knuckle_joint" multiplier="-1"/>
     </joint>
+    <!-- Environment -->
+    <xacro:cube link_name="table" connected_to="world" length="2.00" width="2.00" height="0.25" alpha="0.3">
+      <origin xyz="0 0 -0.125" rpy="0 0 0"/>
+    </xacro:cube>
     <!-- Visual aids for grasping -->
     <link name="finger_tip_closed_point">

Commit message: Get transform working, add calib pose in urdf, add test waypoint, add debug frames

File: src/site_configs/picknik_kinova_satellite_sim/description/picknik_kinova_satellite_sim.xacro (robot description, xacro)
@@ -539,4 +539,10 @@
       <origin xyz="0 0 0.15" rpy="0 0 0"/>
     </joint>
+    <link name="calibration_tool_link"/>
+    <joint name="calibration_tool_joint" type="fixed">
+      <parent link="grasp_link"/>
+      <child link = "calibration_tool_link"/>
+      <origin xyz="0 0 0.15" rpy="${pi/2} 0 0"/>
+    </joint>
     <!-- Camera External -->
     <link name="external_camera_link" />

Commit message: Add calibration tool to urdf

File: src/site_configs/picknik_kinova_satellite_sim/description/picknik_kinova_satellite_sim.xacro (robot description, xacro)
@@ -539,9 +539,21 @@
       <origin xyz="0 0 0.15" rpy="0 0 0"/>
     </joint>
-    <link name="calibration_tool_link"/>
+    <link name="calibration_tool_link">
+      <visual>
+        <geometry>
+          <mesh filename="file://$(find picknik_kinova_satellite_sim)/description/assets/calibration_tool.stl"/>
+        </geometry>
+      </visual>
+    </link>
     <joint name="calibration_tool_joint" type="fixed">
       <parent link="grasp_link"/>
       <child link = "calibration_tool_link"/>
-      <origin xyz="0 0 0.15" rpy="${pi/2} 0 0"/>
+      <origin xyz="0 0 0.019" rpy="0 0 0"/>
+    </joint>
+    <link name="calibration_tool_frame"/>
+    <joint name="calibration_tool_frame_joint" type="fixed">
+      <parent link="calibration_tool_link"/>
+      <child link = "calibration_tool_frame"/>
+      <origin xyz="0 -0.09325 -0.01" rpy="0 ${pi} ${pi}"/>
     </joint>
     <!-- Camera External -->

Commit message: Just use sites for april tag positions

File: src/site_configs/picknik_kinova_satellite_sim/description/picknik_kinova_satellite_sim.xacro (robot description, xacro)
@@ -539,4 +539,23 @@
       <origin xyz="0 0 0.15" rpy="0 0 0"/>
     </joint>
+    <!-- Calibration tool -->
+    <link name="calibration_tool_link">
+      <visual>
+        <geometry>
+          <mesh filename="file://$(find picknik_kinova_satellite_sim)/description/mujoco/assets/calibration_tool.stl"/>
+        </geometry>
+      </visual>
+    </link>
+    <joint name="calibration_tool_joint" type="fixed">
+      <parent link="grasp_link"/>
+      <child link="calibration_tool_link"/>
+      <origin xyz="0 0 0.019" rpy="0 0 0"/>
+    </joint>
+    <link name="calibration_tool_frame"/>
+    <joint name="calibration_tool_frame_joint" type="fixed">
+      <parent link="calibration_tool_link"/>
+      <child link = "calibration_tool_frame"/>
+      <origin xyz="0 -0.09325 -0.01" rpy="0 ${pi} ${pi}"/>
+    </joint>
     <!-- Camera External -->
     <link name="external_camera_link" />
