Commit message: Remove fts, add scene camera, update remaining package names

File: src/site_configs/picknik_006_gen3_hw/description/picknik_006_gen3_hw.xacro (robot description, xacro)
@@ -27,8 +27,7 @@
   <xacro:arg name="gripper_max_force" default="100.0" />
   <xacro:arg name="gripper_com_port" default="/dev/ttyUSB0" />
-  <xacro:arg name="robotiq_fts" default="false" />
-  <xacro:arg name="fts_com_port" default="/dev/ttyUSB1" />
   <!-- Import macros for main hardware components -->
   <xacro:include filename="$(find kortex_description)/robots/kortex_robot.xacro" />
+  <xacro:include filename="$(find picknik_accessories)/descriptions/sensors/realsense_d415.urdf.xacro"/>
   <!-- Import environment macros -->
   <xacro:include filename="$(find picknik_accessories)/descriptions/geometry/cube.urdf.xacro"/>
@@ -41,5 +40,4 @@
   <xacro:arg name="initial_positions_file" default="$(find picknik_006_gen3_hw)/config/initial_positions.yaml"/>
   <xacro:property name="initial_positions_file" default="$(arg initial_positions_file)"/>
-  <xacro:property name="robotiq_fts_property" default="$(arg robotiq_fts)"/>
   <!-- Load the arm -->
   <xacro:load_arm
@@ -71,117 +69,4 @@
   </xacro:load_arm>
   <xacro:property name="gripper_parent_link" value="end_effector_link"/>
-  <!-- If we're using a robotiq fts then add the fts + adapter parts to the urdf -->
-  <xacro:if value="${robotiq_fts_property}">
-    <!-- Adapter that goes between the last link on the kinova and the Robotiq FTS plate -->
-    <link name="fts_coupling_adapter_link">
-      <visual>
-        <origin rpy="0 0 0" xyz="0 0 0"/>
-        <geometry>
-          <cylinder length="0.01115" radius="0.0445"/>
-        </geometry>
-        <material name="green">
-          <color rgba="0 1 0 1"/>
-        </material>
-      </visual>
-      <collision>
-        <origin rpy="0 0 0" xyz="0 0 0"/>
-        <geometry>
-          <cylinder length="0.01115" radius="0.0445"/>
-        </geometry>
-      </collision>
-    </link>
-    <joint name="kinova_fts_coupling_adapter_joint" type="fixed">
-      <parent link="end_effector_link"/>
-      <child link="fts_coupling_adapter_link"/>
-      <origin rpy="0 0 0" xyz="0 0 0.008675"/> <!-- (cylinder length / 2) + 0.0031 offset -->
-    </joint>
-    <!-- Plate that goes between the adapter and the Robotiq FTS -->
-    <link name="fts_coupling_link">
-      <visual>
-        <origin rpy="0 0 0" xyz="0 0 0"/>
-        <geometry>
-          <cylinder length="0.0067" radius="0.0445"/>
-        </geometry>
-        <material name="black">
-          <color rgba="0 0 0 1"/>
-        </material>
-      </visual>
-      <collision>
-        <origin rpy="0 0 0" xyz="0 0 0"/>
-        <geometry>
-          <cylinder length="0.0067" radius="0.0445"/>
-        </geometry>
-      </collision>
-    </link>
-    <joint name="fts_coupling_adapter_fts_coupling_joint" type="fixed">
-      <parent link="fts_coupling_adapter_link"/>
-      <child link="fts_coupling_link"/>
-      <origin rpy="0 0 0" xyz="0 0 0.008925"/> <!-- (cylinder1 length / 2) + (cylinder2 length / 2) -->
-    </joint>
-    <!-- Robotiq FTS -->
-    <link name="fts_link">
-      <visual>
-        <origin rpy="0 0 0" xyz="0 0 0"/>
-        <geometry>
-          <cylinder length="0.0348" radius="0.0445"/>
-        </geometry>
-        <material name="black">
-          <color rgba="0 0 0 1"/>
-        </material>
-      </visual>
-      <collision>
-        <origin rpy="0 0 0" xyz="0 0 0"/>
-        <geometry>
-          <cylinder length="0.0348" radius="0.0445"/>
-        </geometry>
-      </collision>
-    </link>
-    <joint name="fts_plate_fts_joint" type="fixed">
-      <parent link="fts_coupling_link"/>
-      <child link="fts_link"/>
-      <!-- Rotate this link so the FTS link axes are aligned with the FTS hardware -->
-      <origin rpy="0 0 ${pi}" xyz="0 0 0.02075"/> <!-- (cylinder2 length / 2) + (cylinder3 length / 2) -->
-    </joint>
-    <!-- Robotiq gripper controller plate that goes between the FTS and the gripper -->
-    <link name="gripper_plate_link">
-      <visual>
-        <origin rpy="0 0 0" xyz="0 0 0"/>
-        <geometry>
-          <cylinder length="0.0165" radius="0.0375"/>
-        </geometry>
-        <material name="black">
-          <color rgba="0 0 0 1"/>
-        </material>
-      </visual>
-      <collision>
-        <origin rpy="0 0 0" xyz="0 0 0"/>
-        <geometry>
-          <cylinder length="0.0165" radius="0.0375"/>
-        </geometry>
-      </collision>
-    </link>
-    <joint name="fts_gripper_plate_joint" type="fixed">
-      <parent link="fts_link"/>
-      <child link="gripper_plate_link"/>
-      <origin rpy="0 0 0" xyz="0 0 0.02565"/>
-    </joint>
-    <link name="gripper_attachment_link"/>
-    <joint name="gripper_attachment_joint" type="fixed">
-      <parent link="gripper_plate_link"/>
-      <child link="gripper_attachment_link"/>
-      <origin rpy="0 0 ${-pi}" xyz="0 0 0.00515"/> <!-- (cylinder3 length / 2) - 0.0031 offset -->
-    </joint>
-    <!-- Change the gripper parent link if we're using the Robotiq FTS kit -->
-    <xacro:property name="gripper_parent_link" value="gripper_attachment_link"/>
-    <!-- Robotiq FTS ros2_control macro to start the drivers -->
-    <xacro:include filename="$(find robotiq_ft_sensor_description)/urdf/robotiq_fts.ros2_control.xacro" />
-    <xacro:robotiq_fts_ros2_control
-      name=""
-      use_fake_mode="$(arg use_fake_hardware)"
-      max_retries="100"
-      ftdi_id="$(arg fts_com_port)"
-      tf_prefix=""
-    />
-  </xacro:if>
   <!-- change the parent when adding in links in between the gripper and the arm (like a force torque sensor) -->
   <xacro:load_gripper
@@ -250,3 +135,13 @@
     <origin xyz="0 0 0.15" rpy="0 0 0"/>
   </joint>
+    <!-- Camera External -->
+    <link name="external_camera_link" />
+    <joint name="external_camera_joint" type="fixed">
+      <parent link="world" />
+      <child link="external_camera_link" />
+      <origin xyz="-0.3 0.3 1.0" rpy="0 0.5236 0" />
+    </joint>
+    <xacro:realsense_d415 parent="external_camera_link" name="scene_camera">
+      <origin xyz="0 0 0" rpy="0 0 0" />
+    </xacro:realsense_d415>
 </robot>

Commit message: Add hardware description, srdf, control config

File: src/site_configs/picknik_006_gen3_hw/description/picknik_006_gen3_hw.xacro (robot description, xacro)
@@ -6,5 +6,5 @@
   <xacro:arg name="vision" default="false" />
   <xacro:arg name="robot_ip" default="yyy.yyy.yyy.yyy" />
-  <xacro:arg name="gripper" default="robotiq_2f_85" />
+  <xacro:arg name="gripper" default="" />
   <xacro:arg name="username" default="admin" />
   <xacro:arg name="password" default="admin" />
@@ -27,7 +27,8 @@
   <xacro:arg name="gripper_max_force" default="100.0" />
   <xacro:arg name="gripper_com_port" default="/dev/ttyUSB0" />
+  <xacro:arg name="robotiq_fts" default="false" />
+  <xacro:arg name="fts_com_port" default="/dev/ttyUSB1" />
   <!-- Import macros for main hardware components -->
   <xacro:include filename="$(find kortex_description)/robots/kortex_robot.xacro" />
-  <xacro:include filename="$(find picknik_accessories)/descriptions/sensors/realsense_d415.urdf.xacro"/>
   <!-- Import environment macros -->
   <xacro:include filename="$(find picknik_accessories)/descriptions/geometry/cube.urdf.xacro"/>
@@ -40,4 +41,5 @@
   <xacro:arg name="initial_positions_file" default="$(find picknik_006_gen3_hw)/config/initial_positions.yaml"/>
   <xacro:property name="initial_positions_file" default="$(arg initial_positions_file)"/>
+  <xacro:property name="robotiq_fts_property" default="$(arg robotiq_fts)"/>
   <!-- Load the arm -->
   <xacro:load_arm
@@ -69,4 +71,117 @@
   </xacro:load_arm>
   <xacro:property name="gripper_parent_link" value="end_effector_link"/>
+  <!-- If we're using a robotiq fts then add the fts + adapter parts to the urdf -->
+  <xacro:if value="${robotiq_fts_property}">
+    <!-- Adapter that goes between the last link on the kinova and the Robotiq FTS plate -->
+    <link name="fts_coupling_adapter_link">
+      <visual>
+        <origin rpy="0 0 0" xyz="0 0 0"/>
+        <geometry>
+          <cylinder length="0.01115" radius="0.0445"/>
+        </geometry>
+        <material name="green">
+          <color rgba="0 1 0 1"/>
+        </material>
+      </visual>
+      <collision>
+        <origin rpy="0 0 0" xyz="0 0 0"/>
+        <geometry>
+          <cylinder length="0.01115" radius="0.0445"/>
+        </geometry>
+      </collision>
+    </link>
+    <joint name="kinova_fts_coupling_adapter_joint" type="fixed">
+      <parent link="end_effector_link"/>
+      <child link="fts_coupling_adapter_link"/>
+      <origin rpy="0 0 0" xyz="0 0 0.008675"/> <!-- (cylinder length / 2) + 0.0031 offset -->
+    </joint>
+    <!-- Plate that goes between the adapter and the Robotiq FTS -->
+    <link name="fts_coupling_link">
+      <visual>
+        <origin rpy="0 0 0" xyz="0 0 0"/>
+        <geometry>
+          <cylinder length="0.0067" radius="0.0445"/>
+        </geometry>
+        <material name="black">
+          <color rgba="0 0 0 1"/>
+        </material>
+      </visual>
+      <collision>
+        <origin rpy="0 0 0" xyz="0 0 0"/>
+        <geometry>
+          <cylinder length="0.0067" radius="0.0445"/>
+        </geometry>
+      </collision>
+    </link>
+    <joint name="fts_coupling_adapter_fts_coupling_joint" type="fixed">
+      <parent link="fts_coupling_adapter_link"/>
+      <child link="fts_coupling_link"/>
+      <origin rpy="0 0 0" xyz="0 0 0.008925"/> <!-- (cylinder1 length / 2) + (cylinder2 length / 2) -->
+    </joint>
+    <!-- Robotiq FTS -->
+    <link name="fts_link">
+      <visual>
+        <origin rpy="0 0 0" xyz="0 0 0"/>
+        <geometry>
+          <cylinder length="0.0348" radius="0.0445"/>
+        </geometry>
+        <material name="black">
+          <color rgba="0 0 0 1"/>
+        </material>
+      </visual>
+      <collision>
+        <origin rpy="0 0 0" xyz="0 0 0"/>
+        <geometry>
+          <cylinder length="0.0348" radius="0.0445"/>
+        </geometry>
+      </collision>
+    </link>
+    <joint name="fts_plate_fts_joint" type="fixed">
+      <parent link="fts_coupling_link"/>
+      <child link="fts_link"/>
+      <!-- Rotate this link so the FTS link axes are aligned with the FTS hardware -->
+      <origin rpy="0 0 ${pi}" xyz="0 0 0.02075"/> <!-- (cylinder2 length / 2) + (cylinder3 length / 2) -->
+    </joint>
+    <!-- Robotiq gripper controller plate that goes between the FTS and the gripper -->
+    <link name="gripper_plate_link">
+      <visual>
+        <origin rpy="0 0 0" xyz="0 0 0"/>
+        <geometry>
+          <cylinder length="0.0165" radius="0.0375"/>
+        </geometry>
+        <material name="black">
+          <color rgba="0 0 0 1"/>
+        </material>
+      </visual>
+      <collision>
+        <origin rpy="0 0 0" xyz="0 0 0"/>
+        <geometry>
+          <cylinder length="0.0165" radius="0.0375"/>
+        </geometry>
+      </collision>
+    </link>
+    <joint name="fts_gripper_plate_joint" type="fixed">
+      <parent link="fts_link"/>
+      <child link="gripper_plate_link"/>
+      <origin rpy="0 0 0" xyz="0 0 0.02565"/>
+    </joint>
+    <link name="gripper_attachment_link"/>
+    <joint name="gripper_attachment_joint" type="fixed">
+      <parent link="gripper_plate_link"/>
+      <child link="gripper_attachment_link"/>
+      <origin rpy="0 0 ${-pi}" xyz="0 0 0.00515"/> <!-- (cylinder3 length / 2) - 0.0031 offset -->
+    </joint>
+    <!-- Change the gripper parent link if we're using the Robotiq FTS kit -->
+    <xacro:property name="gripper_parent_link" value="gripper_attachment_link"/>
+    <!-- Robotiq FTS ros2_control macro to start the drivers -->
+    <xacro:include filename="$(find robotiq_ft_sensor_description)/urdf/robotiq_fts.ros2_control.xacro" />
+    <xacro:robotiq_fts_ros2_control
+      name=""
+      use_fake_mode="$(arg use_fake_hardware)"
+      max_retries="100"
+      ftdi_id="$(arg fts_com_port)"
+      tf_prefix=""
+    />
+  </xacro:if>
   <!-- change the parent when adding in links in between the gripper and the arm (like a force torque sensor) -->
   <xacro:load_gripper
@@ -135,13 +250,3 @@
     <origin xyz="0 0 0.15" rpy="0 0 0"/>
   </joint>
-    <!-- Camera External -->
-    <link name="external_camera_link" />
-    <joint name="external_camera_joint" type="fixed">
-      <parent link="world" />
-      <child link="external_camera_link" />
-      <origin xyz="-0.3 0.3 1.0" rpy="0 0.5236 0" />
-    </joint>
-    <xacro:realsense_d415 parent="external_camera_link" name="scene_camera">
-      <origin xyz="0 0 0" rpy="0 0 0" />
-    </xacro:realsense_d415>
 </robot>

Commit message: Initial commit, WIP.

File: src/site_configs/picknik_006_gen3_hw/description/picknik_006_gen3_hw.xacro (robot description, xacro)
@@ -250,3 +250,10 @@
     <origin xyz="0 0 0.15" rpy="0 0 0"/>
   </joint>
+  <!-- Add calibration components -->
+  <link name="checkerboard" />
+  <joint name="checkerboard_joint" type="fixed">
+    <parent link="end_effector_link" />
+    <child link="checkerboard" />
+    <origin xyz="0.185 0.037 0.155" rpy="3.142 0.0 3.142" />
+  </joint>
 </robot>

Commit message: Added robot_calibration. WIP. Not working well, abandonded in favor of a Pro calibration workflow.

File: src/site_configs/picknik_006_gen3_hw/description/picknik_006_gen3_hw.xacro (robot description, xacro)
@@ -251,16 +251,57 @@
     <origin xyz="0 0 0.15" rpy="0 0 0"/>
   </joint>
-  <!-- Add calibration components -->
-  <link name="checkerboard" />
-  <joint name="checkerboard_joint" type="fixed">
-    <parent link="end_effector_link" />
-    <child link="checkerboard" />
-    <origin xyz="0.185 0.037 0.155" rpy="3.142 0.0 3.142" />
-  </joint>
   <!-- Scene camera mounted above robot workspace -->
+  <xacro:include filename="$(find picknik_accessories)/descriptions/sensors/extrinsic_calibrated_realsense.urdf.xacro"/>
   <xacro:load_extrinsic_calibrated_realsense
-    name="zed_camera"
+    name="scene_camera_mount"
     parent="base_link"
     model="d415"
     extrinsic_calibration_parameter_file="$(arg scene_camera_calibration_file)" />
+  <!-- Add checkerboard calibration tool -->
+  <link name="calibration_tool">
+    <visual>
+      <geometry>
+        <mesh filename="file://$(find picknik_006_gen3_hw)/description/assets/calibration_tool.dae"/>
+      </geometry>
+    </visual>
+    <collision>
+      <geometry>
+        <mesh filename="file://$(find picknik_006_gen3_hw)/description/assets/calibration_tool.stl"/>
+      </geometry>
+    </collision>
+  </link>
+  <joint name="calibration_tool_joint" type="fixed">
+    <parent link="grasp_link"/>
+    <child link="calibration_tool"/>
+    <origin rpy="0 ${pi} 0" xyz="0.0 -0.0215 0.003"/>
+  </joint>
+  <!-- Add calibration checkerboard frame -->
+  <link name="checkerboard" />
+  <joint name="checkerboard_joint" type="fixed">
+    <parent link="grasp_link" />
+    <child link="checkerboard" />
+    <origin xyz="-0.0619 0.115 0.04657" rpy="3.142 0.0 -1.5708" />
+  </joint>
+  <!-- <link name="camera_wall_link">
+    <visual>
+      <origin xyz="-0.5 0 0" rpy="0 ${pi/2} 0" />
+      <geometry>
+        <cylinder radius="0.02" length="1.0" />
+      </geometry>
+      <material name="Blue">
+        <color rgba="0 0 1.0 0.3" />
+      </material>
+    </visual>
+    <collision>
+      <origin xyz="-0.48 0 0" rpy="0 ${pi/2} 0" />
+      <geometry>
+        <cylinder radius="0.1" length="1.0" />
+      </geometry>
+    </collision>
+  </link>
+  <joint name="camera_wall_joint" type="fixed">
+    <parent link="scene_camera_mount_link" />
+    <child link="camera_wall_link" />
+    <origin xyz="0 0 0" rpy="0 0 0" />
+  </joint> -->
 </robot>

Commit message: Add calibration tool to urdf and add behavior

File: src/site_configs/picknik_006_gen3_hw/description/picknik_006_gen3_hw.xacro (robot description, xacro)
@@ -250,3 +250,21 @@
     <origin xyz="0 0 0.15" rpy="0 0 0"/>
   </joint>
+  <link name="calibration_tool_link">
+    <visual>
+      <geometry>
+        <mesh filename="file://$(find picknik_006_gen3_hw)/description/assets/calibration_tool.stl"/>
+      </geometry>
+    </visual>
+  </link>
+  <joint name="calibration_tool_joint" type="fixed">
+    <parent link="grasp_link"/>
+    <child link = "calibration_tool_link"/>
+    <origin xyz="0 0 0.019" rpy="0 0 0"/>
+  </joint>
+  <link name="calibration_tool_frame"/>
+  <joint name="calibration_tool_frame_joint" type="fixed">
+    <parent link="calibration_tool_link"/>
+    <child link = "calibration_tool_frame"/>
+    <origin xyz="0 -0.09325 -0.01" rpy="0 ${pi} ${pi}"/>
+  </joint>
 </robot>

Commit message: Replace realsense macro with zed urdf. Objective hardcoded offset from optical to mount needs to be updated accordingly.

File: src/site_configs/picknik_006_gen3_hw/description/picknik_006_gen3_hw.xacro (robot description, xacro)
@@ -29,5 +29,4 @@
   <xacro:arg name="robotiq_fts" default="false" />
   <xacro:arg name="fts_com_port" default="/dev/ttyUSB1" />
-  <xacro:arg name="scene_camera_calibration_file" default="package://picknik_006_gen3_hw/objectives/scene_camera_calibration.yaml"/>
   <!-- Import macros for main hardware components -->
   <xacro:include filename="$(find kortex_description)/robots/kortex_robot.xacro" />
@@ -269,9 +268,13 @@
     <origin xyz="0 -0.09325 -0.01" rpy="0 ${pi} ${pi}"/>
   </joint>
-    <!-- Scene camera fixed in robot workspace -->
-  <xacro:include filename="$(find picknik_accessories)/descriptions/sensors/extrinsic_calibrated_realsense.urdf.xacro"/>
-  <xacro:load_extrinsic_calibrated_realsense
-    name="zed_cam"
-    parent="base_link"
-    extrinsic_calibration_parameter_file="$(arg scene_camera_calibration_file)" />
+    <!-- zed camera calibration pose-->
+  <link name="estimated_zed_base_frame" />
+  <joint name="estimated_zed_base_frame_joint" type="fixed">
+    <parent link="base_link" />
+    <child link="estimated_zed_base_frame" />
+    <origin xyz="0.036 0.612 0.374" rpy="0.0099561637429225348 0.066539679824019635 -0.4356580325951358" />
+  </joint>
+  <!-- zed camera URDF-->
+  <xacro:include filename="$(find zed_description)/urdf/zed2i.urdf.xacro"/>
+  <xacro:zed2i parent="estimated_zed_base_frame"/>
 </robot>

Commit message: Updated objectives to use zed left camera.

File: src/site_configs/picknik_006_gen3_hw/description/picknik_006_gen3_hw.xacro (robot description, xacro)
@@ -273,5 +273,6 @@
     <parent link="base_link" />
     <child link="estimated_zed_base_frame" />
-    <origin xyz="0.036 0.612 0.374" rpy="0.0099561637429225348 0.066539679824019635 -0.4356580325951358" />
+    <!-- replace next line with calibrated camera pose (from calibration_pose.txt)  -->
+    <origin xyz=" -0.0364711 0.543233 0.333978" rpy="-0.0155904 0.0406733 -0.543247" />
   </joint>
   <!-- zed camera URDF-->

Commit message: Use zed urdf for camera cal (#8)
* Replace realsense macro with zed urdf. Objective hardcoded offset from optical to mount needs to be updated accordingly.

* Add zed urdf dependency.

* Updated objectives to use zed left camera.

---------

Co-authored-by: David Yackzan <dwyackzan@gmail.com>

File: src/site_configs/picknik_006_gen3_hw/description/picknik_006_gen3_hw.xacro (robot description, xacro)
@@ -29,5 +29,4 @@
   <xacro:arg name="robotiq_fts" default="false" />
   <xacro:arg name="fts_com_port" default="/dev/ttyUSB1" />
-  <xacro:arg name="scene_camera_calibration_file" default="package://picknik_006_gen3_hw/objectives/scene_camera_calibration.yaml"/>
   <!-- Import macros for main hardware components -->
   <xacro:include filename="$(find kortex_description)/robots/kortex_robot.xacro" />
@@ -269,9 +268,14 @@
     <origin xyz="0 -0.09325 -0.01" rpy="0 ${pi} ${pi}"/>
   </joint>
-    <!-- Scene camera fixed in robot workspace -->
-  <xacro:include filename="$(find picknik_accessories)/descriptions/sensors/extrinsic_calibrated_realsense.urdf.xacro"/>
-  <xacro:load_extrinsic_calibrated_realsense
-    name="zed_cam"
-    parent="base_link"
-    extrinsic_calibration_parameter_file="$(arg scene_camera_calibration_file)" />
+    <!-- zed camera calibration pose-->
+  <link name="estimated_zed_base_frame" />
+  <joint name="estimated_zed_base_frame_joint" type="fixed">
+    <parent link="base_link" />
+    <child link="estimated_zed_base_frame" />
+    <!-- replace next line with calibrated camera pose (from calibration_pose.txt)  -->
+    <origin xyz=" -0.0364711 0.543233 0.333978" rpy="-0.0155904 0.0406733 -0.543247" />
+  </joint>
+  <!-- zed camera URDF-->
+  <xacro:include filename="$(find zed_description)/urdf/zed2i.urdf.xacro"/>
+  <xacro:zed2i parent="estimated_zed_base_frame"/>
 </robot>

Commit message: Scale_twist directly from velocity to include the offset. Also updated tags to be the taskboard.

File: src/site_configs/picknik_006_gen3_hw/description/picknik_006_gen3_hw.xacro (robot description, xacro)
@@ -274,5 +274,5 @@
     <child link="estimated_zed_base_frame" />
     <!-- replace next line with calibrated camera pose (from calibration_pose.txt)  -->
-    <origin xyz=" -0.0364711 0.543233 0.333978" rpy="-0.0155904 0.0406733 -0.543247" />
+    <origin xyz=" -0.0364711 0.56 0.32" rpy="-0.0155904 0.0406733 -0.543247" />
   </joint>
   <!-- zed camera URDF-->
